Commit message: Stage 2B: ros2_control mock control loop
- barq.urdf -> barq.urdf.xacro: xmlns:xacro, `mode` arg (mock|gazebo|real),
  <ros2_control> system using mock_components/GenericSystem; 12 joints each with
  a position command interface + position/velocity state interfaces
- ros2_controllers.yaml: joint_state_broadcaster + joint_group_position_controller
- control.launch.py (robot_state_publisher + controller_manager + spawners + optional rviz)
- visualize.launch.py points at the .xacro; setup.py installs config/; package.xml control deps
- Macro params named lower/upper (min/max shadow xacro builtins -> stderr -> launch abort)

Verified headless: 4 nodes up, joint_state_broadcaster + joint_group_position_controller
both active; commanded pose {hips=0, knees=+0.3, ankles=-0.6} reflected in /joint_states.

File: barq_description/urdf/barq.urdf.xacro (robot description, xacro)
@@ -1,4 +1,4 @@
 <?xml version="1.0" ?>
-<robot name="barq">
+<robot name="barq" xmlns:xacro="http://www.ros.org/wiki/xacro">
   <material name="dark_grey">  <color rgba="0.20 0.20 0.20 1.0"/> </material>
   <material name="light_grey"> <color rgba="0.65 0.65 0.65 1.0"/> </material>
@@ -300,3 +300,36 @@
     </inertial>
   </link>
+  <!-- ═══════════════ ros2_control (Stage 2B) ═══════════════ -->
+  <!-- mode: mock (now) | gazebo (2E) | real (Stage 4). Only the <hardware> plugin changes. -->
+  <xacro:arg name="mode" default="mock"/>
+  <xacro:macro name="barq_joint_if" params="name lower upper">
+    <joint name="${name}">
+      <command_interface name="position">
+        <param name="min">${lower}</param>
+        <param name="max">${upper}</param>
+      </command_interface>
+      <state_interface name="position"/>
+      <state_interface name="velocity"/>
+    </joint>
+  </xacro:macro>
+  <ros2_control name="barq_system" type="system">
+    <hardware>
+      <xacro:if value="${'$(arg mode)' == 'mock'}">
+        <plugin>mock_components/GenericSystem</plugin>
+      </xacro:if>
+      <!-- mode=gazebo (Stage 2E) and mode=real (Stage 4) plugins slot in here -->
+    </hardware>
+    <xacro:barq_joint_if name="FL_hip_joint"   lower="-0.785" upper="0.785"/>
+    <xacro:barq_joint_if name="FL_knee_joint"  lower="-1.57"  upper="1.57"/>
+    <xacro:barq_joint_if name="FL_ankle_joint" lower="-1.57"  upper="1.57"/>
+    <xacro:barq_joint_if name="FR_hip_joint"   lower="-0.785" upper="0.785"/>
+    <xacro:barq_joint_if name="FR_knee_joint"  lower="-1.57"  upper="1.57"/>
+    <xacro:barq_joint_if name="FR_ankle_joint" lower="-1.57"  upper="1.57"/>
+    <xacro:barq_joint_if name="RL_hip_joint"   lower="-0.785" upper="0.785"/>
+    <xacro:barq_joint_if name="RL_knee_joint"  lower="-1.57"  upper="1.57"/>
+    <xacro:barq_joint_if name="RL_ankle_joint" lower="-1.57"  upper="1.57"/>
+    <xacro:barq_joint_if name="RR_hip_joint"   lower="-0.785" upper="0.785"/>
+    <xacro:barq_joint_if name="RR_knee_joint"  lower="-1.57"  upper="1.57"/>
+    <xacro:barq_joint_if name="RR_ankle_joint" lower="-1.57"  upper="1.57"/>
+  </ros2_control>
 </robot>

Commit message: Deep crouch: tibia judgment limit -2.2 rad, stand_height 0.115
ST3215s are 360-deg servos - no hard mechanical stops; joint limits are design
judgment (resolves Q-001). Per Aryaman: more femur angle, more tibia fold, narrow.

- Tibia limit -1.57 -> -2.2 (~126 deg) in URDF ankle joints, ros2_control command
  interfaces, robot_params servo map; ik_node clamp now asymmetric [-2.2, 0]
- stand_height 0.16 -> 0.115 (~28% lower); ik_node static stance matches
- New geometric floor: min 2-link reach ~0.094 m at q3=-2.2; stand-step >= ~0.103 m
- Regression test bounds -> [-2.2, 0]; 14 tests pass; xacro clean; check_urdf OK
- D-013: git workflow (push per milestone, author Aryaman Gupta, SSH over 443)

Live-verified: femur +0.93..+0.98, tibia -1.96..-2.08, trot diagonals intact.
Flag: verify link collision at full fold on the physical build before driving
real servos to -2.2 (D-012).

File: barq_description/urdf/barq.urdf.xacro (robot description, xacro)
@@ -71,5 +71,5 @@
     <origin rpy="0 0 0" xyz="0.018944 0.03239997 -0.0999999"/>
     <axis xyz="0 1 0"/>
-    <limit effort="10.0" lower="-1.57" upper="1.57" velocity="5.24"/>
+    <limit effort="10.0" lower="-2.2" upper="1.57" velocity="5.24"/>
     <dynamics damping="0.05" friction="0.0"/>
   </joint>
@@ -141,5 +141,5 @@
     <origin rpy="0 0 0" xyz="0.018944 0.03239997 -0.0999999"/>
     <axis xyz="0 1 0"/>
-    <limit effort="10.0" lower="-1.57" upper="1.57" velocity="5.24"/>
+    <limit effort="10.0" lower="-2.2" upper="1.57" velocity="5.24"/>
     <dynamics damping="0.05" friction="0.0"/>
   </joint>
@@ -211,5 +211,5 @@
     <origin rpy="0 0 0" xyz="0.0189441 -0.03239997 -0.0999999"/>
     <axis xyz="0 1 0"/>
-    <limit effort="10.0" lower="-1.57" upper="1.57" velocity="5.24"/>
+    <limit effort="10.0" lower="-2.2" upper="1.57" velocity="5.24"/>
     <dynamics damping="0.05" friction="0.0"/>
   </joint>
@@ -281,5 +281,5 @@
     <origin rpy="0 0 0" xyz="0.0189441 -0.03239997 -0.0999999"/>
     <axis xyz="0 1 0"/>
-    <limit effort="10.0" lower="-1.57" upper="1.57" velocity="5.24"/>
+    <limit effort="10.0" lower="-2.2" upper="1.57" velocity="5.24"/>
     <dynamics damping="0.05" friction="0.0"/>
   </joint>
@@ -322,14 +322,14 @@
     <xacro:barq_joint_if name="FL_hip_joint"   lower="-0.785" upper="0.785"/>
     <xacro:barq_joint_if name="FL_knee_joint"  lower="-1.57"  upper="1.57"/>
-    <xacro:barq_joint_if name="FL_ankle_joint" lower="-1.57"  upper="1.57"/>
+    <xacro:barq_joint_if name="FL_ankle_joint" lower="-2.2"   upper="1.57"/>
     <xacro:barq_joint_if name="FR_hip_joint"   lower="-0.785" upper="0.785"/>
     <xacro:barq_joint_if name="FR_knee_joint"  lower="-1.57"  upper="1.57"/>
-    <xacro:barq_joint_if name="FR_ankle_joint" lower="-1.57"  upper="1.57"/>
+    <xacro:barq_joint_if name="FR_ankle_joint" lower="-2.2"   upper="1.57"/>
     <xacro:barq_joint_if name="RL_hip_joint"   lower="-0.785" upper="0.785"/>
     <xacro:barq_joint_if name="RL_knee_joint"  lower="-1.57"  upper="1.57"/>
-    <xacro:barq_joint_if name="RL_ankle_joint" lower="-1.57"  upper="1.57"/>
+    <xacro:barq_joint_if name="RL_ankle_joint" lower="-2.2"   upper="1.57"/>
     <xacro:barq_joint_if name="RR_hip_joint"   lower="-0.785" upper="0.785"/>
     <xacro:barq_joint_if name="RR_knee_joint"  lower="-1.57"  upper="1.57"/>
-    <xacro:barq_joint_if name="RR_ankle_joint" lower="-1.57"  upper="1.57"/>
+    <xacro:barq_joint_if name="RR_ankle_joint" lower="-2.2"   upper="1.57"/>
   </ros2_control>
 </robot>

Commit message: Stage 2E: BARQ walks in Gazebo physics (exact kinematics, head-first)
Infrastructure:
- Dockerfile: OSRF repo + slim gz set (ros-gz-sim, ros-gz-bridge, ign-ros2-control;
  the ros-gz metapackage pulls libopencv-dev which collides with dustynv CUDA opencv)
- barq.urdf.xacro: mode:=gazebo (ign_ros2_control hardware + system plugin); collisions
  reduced to body box + 4 foot contact spheres at the kinematic foot points
- barq_sim: offline barq_world.sdf; sim.launch.py (gz server/GUI, spawn, /clock bridge,
  spawners, gait:=true)

Review-driven fixes (25-agent adversarial review: 3 confirmed, 18 refuted):
- EXACT URDF-true leg kinematics (fk_exact/ik_exact): knee-x +-0.01744 front/rear,
  femur in-plane L2P at fixed angle A2, lateral 0.0754692, URDF-true q2 sign. The old
  idealized model erred up to 3.4 cm at the front feet (asymmetric) - the root cause of
  the reversed walk direction and an 11 mm height anomaly. Locked by
  test_exact_kinematics.py (FK == raw URDF chain composition < 1e-12; IK round-trip)
- Startup: initial_value = exact stance (0, 1.047531, -1.928768) on all 12 joints,
  spawn z 0.17 - no more collapse + first-command snap
- Swing clearance: gait stand 0.13 / step 0.02; gait_planner forward_sign param

Physics verified (ign model --pose): settle z 0.141779 vs 0.142 predicted (0.2 mm),
zero startup transient; cmd_vel +x walks -0.376 m in ~8 s toward -X = HEAD-FIRST
(correct; was tail-first). 19 unit tests pass.

File: barq_description/urdf/barq.urdf.xacro (robot description, xacro)
@@ -34,8 +34,4 @@
       <material name="dark_grey"/>
     </visual>
-    <collision>
-      <origin rpy="3.14159265358979 0 -1.5708" xyz="0 0 0"/>
-      <geometry><mesh filename="package://barq_description/meshes/coxa.dae" scale="1 1 1"/></geometry>
-    </collision>
     <inertial>
       <mass value="0.077"/>
@@ -57,8 +53,4 @@
       <material name="dark_grey"/>
     </visual>
-    <collision>
-      <origin rpy="0 0 -1.5708" xyz="0 0 0"/>
-      <geometry><mesh filename="package://barq_description/meshes/mid.dae" scale="1 1 1"/></geometry>
-    </collision>
     <inertial>
       <mass value="0.05"/>
@@ -80,7 +72,8 @@
       <material name="dark_grey"/>
     </visual>
-    <collision>
-      <origin rpy="0 0 -1.5708" xyz="0 0 0"/>
-      <geometry><mesh filename="package://barq_description/meshes/foot.dae" scale="1 1 1"/></geometry>
+    <!-- Contact sphere at the kinematic foot point (mesh collisions are unstable/slow in sim) -->
+    <collision>
+      <origin rpy="0 0 0" xyz="0 0 -0.1"/>
+      <geometry><sphere radius="0.012"/></geometry>
     </collision>
     <inertial>
@@ -104,8 +97,4 @@
       <material name="dark_grey"/>
     </visual>
-    <collision>
-      <origin rpy="0 0 -1.5708" xyz="0 0 0"/>
-      <geometry><mesh filename="package://barq_description/meshes/coxa.dae" scale="1 1 1"/></geometry>
-    </collision>
     <inertial>
       <mass value="0.077"/>
@@ -127,8 +116,4 @@
       <material name="dark_grey"/>
     </visual>
-    <collision>
-      <origin rpy="0 0 -1.5708" xyz="0 0 0"/>
-      <geometry><mesh filename="package://barq_description/meshes/mid.dae" scale="1 1 1"/></geometry>
-    </collision>
     <inertial>
       <mass value="0.05"/>
@@ -150,7 +135,8 @@
       <material name="dark_grey"/>
     </visual>
-    <collision>
-      <origin rpy="0 0 -1.5708" xyz="0 0 0"/>
-      <geometry><mesh filename="package://barq_description/meshes/foot.dae" scale="1 1 1"/></geometry>
+    <!-- Contact sphere at the kinematic foot point (mesh collisions are unstable/slow in sim) -->
+    <collision>
+      <origin rpy="0 0 0" xyz="0 0 -0.1"/>
+      <geometry><sphere radius="0.012"/></geometry>
     </collision>
     <inertial>
@@ -174,8 +160,4 @@
       <material name="dark_grey"/>
     </visual>
-    <collision>
-      <origin rpy="0 0 1.5708" xyz="0 0 0"/>
-      <geometry><mesh filename="package://barq_description/meshes/coxa.dae" scale="1 1 1"/></geometry>
-    </collision>
     <inertial>
       <mass value="0.077"/>
@@ -197,8 +179,4 @@
       <material name="dark_grey"/>
     </visual>
-    <collision>
-      <origin rpy="0 0 -1.5708" xyz="0 0 0"/>
-      <geometry><mesh filename="package://barq_description/meshes/mid_rev.dae" scale="1 1 1"/></geometry>
-    </collision>
     <inertial>
       <mass value="0.05"/>
@@ -220,7 +198,8 @@
       <material name="dark_grey"/>
     </visual>
-    <collision>
-      <origin rpy="0 0 -1.5708" xyz="0 0 0"/>
-      <geometry><mesh filename="package://barq_description/meshes/foot_rev.dae" scale="1 1 1"/></geometry>
+    <!-- Contact sphere at the kinematic foot point (mesh collisions are unstable/slow in sim) -->
+    <collision>
+      <origin rpy="0 0 0" xyz="0 0 -0.1"/>
+      <geometry><sphere radius="0.012"/></geometry>
     </collision>
     <inertial>
@@ -244,8 +223,4 @@
       <material name="dark_grey"/>
     </visual>
-    <collision>
-      <origin rpy="3.14159265358979 0 1.5708" xyz="0 0 0"/>
-      <geometry><mesh filename="package://barq_description/meshes/coxa.dae" scale="1 1 1"/></geometry>
-    </collision>
     <inertial>
       <mass value="0.077"/>
@@ -267,8 +242,4 @@
       <material name="dark_grey"/>
     </visual>
-    <collision>
-      <origin rpy="0 0 -1.5708" xyz="0 0 0"/>
-      <geometry><mesh filename="package://barq_description/meshes/mid_rev.dae" scale="1 1 1"/></geometry>
-    </collision>
     <inertial>
       <mass value="0.05"/>
@@ -290,7 +261,8 @@
       <material name="dark_grey"/>
     </visual>
-    <collision>
-      <origin rpy="0 0 -1.5708" xyz="0 0 0"/>
-      <geometry><mesh filename="package://barq_description/meshes/foot_rev.dae" scale="1 1 1"/></geometry>
+    <!-- Contact sphere at the kinematic foot point (mesh collisions are unstable/slow in sim) -->
+    <collision>
+      <origin rpy="0 0 0" xyz="0 0 -0.1"/>
+      <geometry><sphere radius="0.012"/></geometry>
     </collision>
     <inertial>
@@ -303,5 +275,7 @@
   <!-- mode: mock (now) | gazebo (2E) | real (Stage 4). Only the <hardware> plugin changes. -->
   <xacro:arg name="mode" default="mock"/>
-  <xacro:macro name="barq_joint_if" params="name lower upper">
+  <!-- init = startup joint position (the exact-model standing stance, stand_height 0.13):
+       prevents the spawn collapse + first-command snap found in the 2E review. -->
+  <xacro:macro name="barq_joint_if" params="name lower upper init">
     <joint name="${name}">
       <command_interface name="position">
@@ -309,5 +283,7 @@
         <param name="max">${upper}</param>
       </command_interface>
-      <state_interface name="position"/>
+      <state_interface name="position">
+        <param name="initial_value">${init}</param>
+      </state_interface>
       <state_interface name="velocity"/>
     </joint>
@@ -318,18 +294,33 @@
         <plugin>mock_components/GenericSystem</plugin>
       </xacro:if>
-      <!-- mode=gazebo (Stage 2E) and mode=real (Stage 4) plugins slot in here -->
+      <xacro:if value="${'$(arg mode)' == 'gazebo'}">
+        <plugin>ign_ros2_control/IgnitionSystem</plugin>
+      </xacro:if>
+      <!-- mode=real (Stage 4) plugin slots in here -->
     </hardware>
-    <xacro:barq_joint_if name="FL_hip_joint"   lower="-0.785" upper="0.785"/>
-    <xacro:barq_joint_if name="FL_knee_joint"  lower="-1.57"  upper="1.57"/>
-    <xacro:barq_joint_if name="FL_ankle_joint" lower="-2.2"   upper="1.57"/>
-    <xacro:barq_joint_if name="FR_hip_joint"   lower="-0.785" upper="0.785"/>
-    <xacro:barq_joint_if name="FR_knee_joint"  lower="-1.57"  upper="1.57"/>
-    <xacro:barq_joint_if name="FR_ankle_joint" lower="-2.2"   upper="1.57"/>
-    <xacro:barq_joint_if name="RL_hip_joint"   lower="-0.785" upper="0.785"/>
-    <xacro:barq_joint_if name="RL_knee_joint"  lower="-1.57"  upper="1.57"/>
-    <xacro:barq_joint_if name="RL_ankle_joint" lower="-2.2"   upper="1.57"/>
-    <xacro:barq_joint_if name="RR_hip_joint"   lower="-0.785" upper="0.785"/>
-    <xacro:barq_joint_if name="RR_knee_joint"  lower="-1.57"  upper="1.57"/>
-    <xacro:barq_joint_if name="RR_ankle_joint" lower="-2.2"   upper="1.57"/>
+    <xacro:barq_joint_if name="FL_hip_joint"   lower="-0.785" upper="0.785" init="0.0"/>
+    <xacro:barq_joint_if name="FL_knee_joint"  lower="-1.57"  upper="1.57" init="1.047531"/>
+    <xacro:barq_joint_if name="FL_ankle_joint" lower="-2.2"   upper="1.57" init="-1.928768"/>
+    <xacro:barq_joint_if name="FR_hip_joint"   lower="-0.785" upper="0.785" init="0.0"/>
+    <xacro:barq_joint_if name="FR_knee_joint"  lower="-1.57"  upper="1.57" init="1.047531"/>
+    <xacro:barq_joint_if name="FR_ankle_joint" lower="-2.2"   upper="1.57" init="-1.928768"/>
+    <xacro:barq_joint_if name="RL_hip_joint"   lower="-0.785" upper="0.785" init="0.0"/>
+    <xacro:barq_joint_if name="RL_knee_joint"  lower="-1.57"  upper="1.57" init="1.047531"/>
+    <xacro:barq_joint_if name="RL_ankle_joint" lower="-2.2"   upper="1.57" init="-1.928768"/>
+    <xacro:barq_joint_if name="RR_hip_joint"   lower="-0.785" upper="0.785" init="0.0"/>
+    <xacro:barq_joint_if name="RR_knee_joint"  lower="-1.57"  upper="1.57" init="1.047531"/>
+    <xacro:barq_joint_if name="RR_ankle_joint" lower="-2.2"   upper="1.57" init="-1.928768"/>
   </ros2_control>
+  <!-- ═══════════════ Gazebo (Stage 2E, mode:=gazebo) ═══════════════ -->
+  <xacro:if value="${'$(arg mode)' == 'gazebo'}">
+    <gazebo>
+      <plugin filename="ign_ros2_control-system" name="ign_ros2_control::IgnitionROS2ControlPlugin">
+        <parameters>$(find barq_bringup)/config/ros2_controllers.yaml</parameters>
+      </plugin>
+    </gazebo>
+    <gazebo reference="FL_tibia_link"><mu1>0.9</mu1><mu2>0.9</mu2></gazebo>
+    <gazebo reference="FR_tibia_link"><mu1>0.9</mu1><mu2>0.9</mu2></gazebo>
+    <gazebo reference="RL_tibia_link"><mu1>0.9</mu1><mu2>0.9</mu2></gazebo>
+    <gazebo reference="RR_tibia_link"><mu1>0.9</mu1><mu2>0.9</mu2></gazebo>
+  </xacro:if>
 </robot>
