Commit message: Measured masses + real ST3215 torque caps (2.94 Nm) in the model
Measured by Aryaman (servos/fasteners included): body 1.42 kg, coxa 73.3 g,
femur 153.6 g, tibia 30 g -> total 2.448 kg (femur was 3x underestimated).
Effort limit 10.0 -> 2.94 N.m (30 kg.cm mechanical peak) on all 12 joints -
enforced by ign_ros2_control in physics. Inertia tensors recomputed from
primitive shapes at measured masses (placeholders replaced). robot_params:
body mass, link_masses, actuators section (ST3215, 2.94 N.m, 5.24 rad/s).

Physics A/B: settle z 0.141779 unchanged, level; walk +0.523 m/10 s (was
+0.44 - more friction authority); servos hold the real robot with ~5-10x
stance margin.

File: barq_description/urdf/barq.urdf.xacro (robot description, xacro)
@@ -14,8 +14,10 @@
       <geometry><box size="0.258 0.117 0.085"/></geometry>
     </collision>
-    <inertial>
-      <mass value="0.95"/>
+    <!-- Measured 2026-06-11 (Aryaman): incl. electronics/fasteners. Inertia: solid box
+         0.258 x 0.117 x 0.085 at the measured mass. -->
+    <inertial>
+      <mass value="1.42"/>
       <origin rpy="0 0 0" xyz="0 0 0"/>
-      <inertia ixx="3.0e-3" ixy="0" ixz="0" iyy="5.5e-3" iyz="0" izz="6.5e-3"/>
+      <inertia ixx="2.47e-3" ixy="0" ixz="0" iyy="8.73e-3" iyz="0" izz="9.50e-3"/>
     </inertial>
   </link>
@@ -25,5 +27,5 @@
     <origin rpy="0 0 0" xyz="0.108484 0.0171913 0.00022012"/>
     <axis xyz="1 0 0"/>
-    <limit effort="10.0" lower="-0.785" upper="0.785" velocity="5.24"/>
+    <limit effort="2.94" lower="-0.785" upper="0.785" velocity="5.24"/>
     <dynamics damping="0.05" friction="0.0"/>
   </joint>
@@ -35,7 +37,7 @@
     </visual>
     <inertial>
-      <mass value="0.077"/>
+      <mass value="0.0733"/>
       <origin rpy="0 0 0" xyz="0.00872 0.0215346 0"/>
-      <inertia ixx="1.0e-5" ixy="0" ixz="0" iyy="1.0e-4" iyz="0" izz="1.0e-4"/>
+      <inertia ixx="3.2e-5" ixy="0" ixz="0" iyy="2.0e-5" iyz="0" izz="3.2e-5"/>
     </inertial>
   </link>
@@ -44,5 +46,5 @@
     <origin rpy="0 0 0" xyz="0.01744 0.0430692 0"/>
     <axis xyz="0 1 0"/>
-    <limit effort="10.0" lower="-1.57" upper="1.57" velocity="5.24"/>
+    <limit effort="2.94" lower="-1.57" upper="1.57" velocity="5.24"/>
     <dynamics damping="0.05" friction="0.0"/>
   </joint>
@@ -54,7 +56,7 @@
     </visual>
     <inertial>
-      <mass value="0.05"/>
+      <mass value="0.1536"/>
       <origin rpy="0 0 0" xyz="0.009472 0.01769995 -0.04999995"/>
-      <inertia ixx="1.0e-4" ixy="0" ixz="0" iyy="1.0e-4" iyz="0" izz="1.0e-5"/>
+      <inertia ixx="1.7e-4" ixy="0" ixz="0" iyy="1.6e-4" iyz="0" izz="5.3e-5"/>
     </inertial>
   </link>
@@ -63,5 +65,5 @@
     <origin rpy="0 0 0" xyz="0.018944 0.03239997 -0.0999999"/>
     <axis xyz="0 1 0"/>
-    <limit effort="10.0" lower="-2.2" upper="1.57" velocity="5.24"/>
+    <limit effort="2.94" lower="-2.2" upper="1.57" velocity="5.24"/>
     <dynamics damping="0.05" friction="0.0"/>
   </joint>
@@ -78,7 +80,7 @@
     </collision>
     <inertial>
-      <mass value="0.05"/>
+      <mass value="0.030"/>
       <origin rpy="0 0 0" xyz="0 0 -0.04999995"/>
-      <inertia ixx="1.0e-4" ixy="0" ixz="0" iyy="1.0e-4" iyz="0" izz="1.0e-5"/>
+      <inertia ixx="3.3e-5" ixy="0" ixz="0" iyy="3.1e-5" iyz="0" izz="3.3e-6"/>
     </inertial>
   </link>
@@ -88,5 +90,5 @@
     <origin rpy="0 0 0" xyz="-0.108371 0.0167905 0.00022176"/>
     <axis xyz="1 0 0"/>
-    <limit effort="10.0" lower="-0.785" upper="0.785" velocity="5.24"/>
+    <limit effort="2.94" lower="-0.785" upper="0.785" velocity="5.24"/>
     <dynamics damping="0.05" friction="0.0"/>
   </joint>
@@ -98,7 +100,7 @@
     </visual>
     <inertial>
-      <mass value="0.077"/>
+      <mass value="0.0733"/>
       <origin rpy="0 0 0" xyz="-0.00872 0.0215346 0"/>
-      <inertia ixx="1.0e-5" ixy="0" ixz="0" iyy="1.0e-4" iyz="0" izz="1.0e-4"/>
+      <inertia ixx="3.2e-5" ixy="0" ixz="0" iyy="2.0e-5" iyz="0" izz="3.2e-5"/>
     </inertial>
   </link>
@@ -107,5 +109,5 @@
     <origin rpy="0 0 0" xyz="-0.01744 0.0430692 0"/>
     <axis xyz="0 1 0"/>
-    <limit effort="10.0" lower="-1.57" upper="1.57" velocity="5.24"/>
+    <limit effort="2.94" lower="-1.57" upper="1.57" velocity="5.24"/>
     <dynamics damping="0.05" friction="0.0"/>
   </joint>
@@ -117,7 +119,7 @@
     </visual>
     <inertial>
-      <mass value="0.05"/>
+      <mass value="0.1536"/>
       <origin rpy="0 0 0" xyz="0.009472 0.01769995 -0.04999995"/>
-      <inertia ixx="1.0e-4" ixy="0" ixz="0" iyy="1.0e-4" iyz="0" izz="1.0e-5"/>
+      <inertia ixx="1.7e-4" ixy="0" ixz="0" iyy="1.6e-4" iyz="0" izz="5.3e-5"/>
     </inertial>
   </link>
@@ -126,5 +128,5 @@
     <origin rpy="0 0 0" xyz="0.018944 0.03239997 -0.0999999"/>
     <axis xyz="0 1 0"/>
-    <limit effort="10.0" lower="-2.2" upper="1.57" velocity="5.24"/>
+    <limit effort="2.94" lower="-2.2" upper="1.57" velocity="5.24"/>
     <dynamics damping="0.05" friction="0.0"/>
   </joint>
@@ -141,7 +143,7 @@
     </collision>
     <inertial>
-      <mass value="0.05"/>
+      <mass value="0.030"/>
       <origin rpy="0 0 0" xyz="0 0 -0.04999995"/>
-      <inertia ixx="1.0e-4" ixy="0" ixz="0" iyy="1.0e-4" iyz="0" izz="1.0e-5"/>
+      <inertia ixx="3.3e-5" ixy="0" ixz="0" iyy="3.1e-5" iyz="0" izz="3.3e-6"/>
     </inertial>
   </link>
@@ -151,5 +153,5 @@
     <origin rpy="0 0 0" xyz="0.108484 -0.0148092 0.00022176"/>
     <axis xyz="1 0 0"/>
-    <limit effort="10.0" lower="-0.785" upper="0.785" velocity="5.24"/>
+    <limit effort="2.94" lower="-0.785" upper="0.785" velocity="5.24"/>
     <dynamics damping="0.05" friction="0.0"/>
   </joint>
@@ -161,7 +163,7 @@
     </visual>
     <inertial>
-      <mass value="0.077"/>
+      <mass value="0.0733"/>
       <origin rpy="0 0 0" xyz="0.00872 -0.0215346 0"/>
-      <inertia ixx="1.0e-5" ixy="0" ixz="0" iyy="1.0e-4" iyz="0" izz="1.0e-4"/>
+      <inertia ixx="3.2e-5" ixy="0" ixz="0" iyy="2.0e-5" iyz="0" izz="3.2e-5"/>
     </inertial>
   </link>
@@ -170,5 +172,5 @@
     <origin rpy="0 0 0" xyz="0.01744 -0.0430692 0"/>
     <axis xyz="0 1 0"/>
-    <limit effort="10.0" lower="-1.57" upper="1.57" velocity="5.24"/>
+    <limit effort="2.94" lower="-1.57" upper="1.57" velocity="5.24"/>
     <dynamics damping="0.05" friction="0.0"/>
   </joint>
@@ -180,7 +182,7 @@
     </visual>
     <inertial>
-      <mass value="0.05"/>
+      <mass value="0.1536"/>
       <origin rpy="0 0 0" xyz="0.00947205 -0.01769995 -0.04999995"/>
-      <inertia ixx="1.0e-4" ixy="0" ixz="0" iyy="1.0e-4" iyz="0" izz="1.0e-5"/>
+      <inertia ixx="1.7e-4" ixy="0" ixz="0" iyy="1.6e-4" iyz="0" izz="5.3e-5"/>
     </inertial>
   </link>
@@ -189,5 +191,5 @@
     <origin rpy="0 0 0" xyz="0.0189441 -0.03239997 -0.0999999"/>
     <axis xyz="0 1 0"/>
-    <limit effort="10.0" lower="-2.2" upper="1.57" velocity="5.24"/>
+    <limit effort="2.94" lower="-2.2" upper="1.57" velocity="5.24"/>
     <dynamics damping="0.05" friction="0.0"/>
   </joint>
@@ -204,7 +206,7 @@
     </collision>
     <inertial>
-      <mass value="0.05"/>
+      <mass value="0.030"/>
       <origin rpy="0 0 0" xyz="0 0 -0.04999995"/>
-      <inertia ixx="1.0e-4" ixy="0" ixz="0" iyy="1.0e-4" iyz="0" izz="1.0e-5"/>
+      <inertia ixx="3.3e-5" ixy="0" ixz="0" iyy="3.1e-5" iyz="0" izz="3.3e-6"/>
     </inertial>
   </link>
@@ -214,5 +216,5 @@
     <origin rpy="0 0 0" xyz="-0.108371 -0.01521 0.00022012"/>
     <axis xyz="1 0 0"/>
-    <limit effort="10.0" lower="-0.785" upper="0.785" velocity="5.24"/>
+    <limit effort="2.94" lower="-0.785" upper="0.785" velocity="5.24"/>
     <dynamics damping="0.05" friction="0.0"/>
   </joint>
@@ -224,7 +226,7 @@
     </visual>
     <inertial>
-      <mass value="0.077"/>
+      <mass value="0.0733"/>
       <origin rpy="0 0 0" xyz="-0.00872 -0.0215346 0"/>
-      <inertia ixx="1.0e-5" ixy="0" ixz="0" iyy="1.0e-4" iyz="0" izz="1.0e-4"/>
+      <inertia ixx="3.2e-5" ixy="0" ixz="0" iyy="2.0e-5" iyz="0" izz="3.2e-5"/>
     </inertial>
   </link>
@@ -233,5 +235,5 @@
     <origin rpy="0 0 0" xyz="-0.01744 -0.0430692 0"/>
     <axis xyz="0 1 0"/>
-    <limit effort="10.0" lower="-1.57" upper="1.57" velocity="5.24"/>
+    <limit effort="2.94" lower="-1.57" upper="1.57" velocity="5.24"/>
     <dynamics damping="0.05" friction="0.0"/>
   </joint>
@@ -243,7 +245,7 @@
     </visual>
     <inertial>
-      <mass value="0.05"/>
+      <mass value="0.1536"/>
       <origin rpy="0 0 0" xyz="0.00947205 -0.01769995 -0.04999995"/>
-      <inertia ixx="1.0e-4" ixy="0" ixz="0" iyy="1.0e-4" iyz="0" izz="1.0e-5"/>
+      <inertia ixx="1.7e-4" ixy="0" ixz="0" iyy="1.6e-4" iyz="0" izz="5.3e-5"/>
     </inertial>
   </link>
@@ -252,5 +254,5 @@
     <origin rpy="0 0 0" xyz="0.0189441 -0.03239997 -0.0999999"/>
     <axis xyz="0 1 0"/>
-    <limit effort="10.0" lower="-2.2" upper="1.57" velocity="5.24"/>
+    <limit effort="2.94" lower="-2.2" upper="1.57" velocity="5.24"/>
     <dynamics damping="0.05" friction="0.0"/>
   </joint>
@@ -267,7 +269,7 @@
     </collision>
     <inertial>
-      <mass value="0.05"/>
+      <mass value="0.030"/>
       <origin rpy="0 0 0" xyz="0 0 -0.04999995"/>
-      <inertia ixx="1.0e-4" ixy="0" ixz="0" iyy="1.0e-4" iyz="0" izz="1.0e-5"/>
+      <inertia ixx="3.3e-5" ixy="0" ixz="0" iyy="3.1e-5" iyz="0" izz="3.3e-6"/>
     </inertial>
   </link>

Commit message: Sim perception: 2D lidar + slam_toolbox map the room in Gazebo
- URDF: laser link (47 g, aft deck, -4.5 deg counter-wedge) + gpu_lidar
  (360 deg / 2160 samples / 25 m, STL-27L-class; purchase deferred Q-015) +
  ground-truth OdometryPublisher - gazebo mode only
- World: Sensors system (ogre2, headless EGL - works on Tegra) + 8x6 m walled
  room with pillars (empty world maps nothing - features required)
- Launch: /scan + /odom bridges, slam:=true (slam_toolbox + barq_slam.yaml),
  odom_tf node with FORCED frame names (gz model-prefixes TF frames, which
  silently broke slam_toolbox's odom->laser chain)
- Image: + slam-toolbox, laser-filters; viewer config barq_slam.rviz

Verified: odom->laser rotation ~0 (counter-wedge cancels stance pitch exactly);
scan 7-9.7 Hz; map 161x121 @ 0.05 m = the room (1127 occupied / 16898 free)
after one driven lap; map->odom TF live. RTF ~41% under full perception load.

File: barq_description/urdf/barq.urdf.xacro (robot description, xacro)
@@ -22,4 +22,24 @@
     </inertial>
   </link>
+  <!-- ═══════════════ LIDAR (STL-27L-class 2D, Q-015: purchase deferred, sim-first) ═══════════
+       Aft-of-center deck mount (nose reserved for a future depth camera). Pitched -4.5 deg to
+       counter the nose-down stance trim (D-016) so the scan plane is level at nominal stance.
+       Mass modelled so dynamics/RL train on the robot that will exist. -->
+  <link name="laser">
+    <visual>
+      <origin rpy="0 0 0" xyz="0 0 0"/>
+      <geometry><cylinder radius="0.019" length="0.035"/></geometry>
+      <material name="dark_grey"/>
+    </visual>
+    <inertial>
+      <mass value="0.047"/>
+      <origin rpy="0 0 0" xyz="0 0 0"/>
+      <inertia ixx="1.0e-5" ixy="0" ixz="0" iyy="1.0e-5" iyz="0" izz="8.5e-6"/>
+    </inertial>
+  </link>
+  <joint name="laser_joint" type="fixed">
+    <parent link="base_link"/>    <child link="laser"/>
+    <origin rpy="0 -0.0785 0" xyz="-0.04 0 0.066"/>
+  </joint>
   <!-- ═══════════════ FL LEG ═══════════════ -->
   <joint name="FL_hip_joint" type="revolute">
@@ -326,4 +346,38 @@
     <gazebo reference="RL_tibia_link"><mu1>0.9</mu1><mu2>0.9</mu2></gazebo>
     <gazebo reference="RR_tibia_link"><mu1>0.9</mu1><mu2>0.9</mu2></gazebo>
+    <!-- 2D lidar (STL-27L-class: 360 deg, 25 m, 21.6 kHz -> 2160 samples @ 10 Hz).
+         frame/topic chosen for zero-config parity with the real driver (frame 'laser', /scan). -->
+    <gazebo reference="laser">
+      <sensor name="lidar2d" type="gpu_lidar">
+        <topic>scan</topic>
+        <update_rate>10</update_rate>
+        <ignition_frame_id>laser</ignition_frame_id>
+        <lidar>
+          <scan>
+            <horizontal>
+              <samples>2160</samples>
+              <resolution>1</resolution>
+              <min_angle>-3.14159</min_angle>
+              <max_angle>3.14159</max_angle>
+            </horizontal>
+          </scan>
+          <range><min>0.15</min><max>25.0</max><resolution>0.01</resolution></range>
+          <noise><type>gaussian</type><mean>0.0</mean><stddev>0.02</stddev></noise>
+        </lidar>
+        <always_on>1</always_on>
+        <visualize>false</visualize>
+      </sensor>
+    </gazebo>
+    <!-- Ground-truth odometry STOPGAP for SLAM (slam_toolbox needs odom->base_link TF; real
+         legged odometry comes with the state estimator). Makes SLAM look artificially clean. -->
+    <gazebo>
+      <plugin filename="ignition-gazebo-odometry-publisher-system"
+              name="ignition::gazebo::systems::OdometryPublisher">
+        <odom_frame>odom</odom_frame>
+        <robot_base_frame>base_link</robot_base_frame>
+        <odom_publish_frequency>50</odom_publish_frequency>
+        <dimensions>3</dimensions>
+      </plugin>
+    </gazebo>
   </xacro:if>
 </robot>

Commit message: Sim made ST3215-true: engine-verified envelope, k=60 servo stiffness (vendored plugin patch), swing-drag fix (~60% realized speed)
- URDF velocity caps 5.24->4.71 rad/s (Waveshare spec); envelope verified at engine
  level via 'ign sdf -p' (effort/velocity/mu x12)
- Found+patched ign_ros2_control 0.7.x param-ordering bug: node constructed before
  <parameters> reach rcl global args -> position_proportional_gain unreachable.
  Vendored external/gz_ros2_control (BARQ.patch, PROVENANCE.md); launch shadows
  /opt via IGN_GAZEBO_SYSTEM_PLUGIN_PATH. k=10->60/s: step rise 200->50ms,
  trot tracking 55.4->17.8 mrad mean RMS (bag-based metric, starvation-immune)
- Q-013 solved: mu-invariant speed deficit (0.25/0.5/0.9 sweep) = swing-foot drag;
  front clearance reach-capped at 20mm. Smoothstep swing + duty 0.6 -> ~60%
  realized; duty 0.55 dead straight (Q-016 tracks yaw-vs-duty)
- New: diagnostics/sim_actuation_probe.py, sim_walk_metric.py, analyze_track_bag.py;
  launch args foot_mu/gait_duty/gait_period; D-018, D-019; research log 2f

File: barq_description/urdf/barq.urdf.xacro (robot description, xacro)
@@ -47,5 +47,5 @@
     <origin rpy="0 0 0" xyz="0.108484 0.0171913 0.00022012"/>
     <axis xyz="1 0 0"/>
-    <limit effort="2.94" lower="-0.785" upper="0.785" velocity="5.24"/>
+    <limit effort="2.94" lower="-0.785" upper="0.785" velocity="4.71"/>
     <dynamics damping="0.05" friction="0.0"/>
   </joint>
@@ -66,5 +66,5 @@
     <origin rpy="0 0 0" xyz="0.01744 0.0430692 0"/>
     <axis xyz="0 1 0"/>
-    <limit effort="2.94" lower="-1.57" upper="1.57" velocity="5.24"/>
+    <limit effort="2.94" lower="-1.57" upper="1.57" velocity="4.71"/>
     <dynamics damping="0.05" friction="0.0"/>
   </joint>
@@ -85,5 +85,5 @@
     <origin rpy="0 0 0" xyz="0.018944 0.03239997 -0.0999999"/>
     <axis xyz="0 1 0"/>
-    <limit effort="2.94" lower="-2.2" upper="1.57" velocity="5.24"/>
+    <limit effort="2.94" lower="-2.2" upper="1.57" velocity="4.71"/>
     <dynamics damping="0.05" friction="0.0"/>
   </joint>
@@ -110,5 +110,5 @@
     <origin rpy="0 0 0" xyz="-0.108371 0.0167905 0.00022176"/>
     <axis xyz="1 0 0"/>
-    <limit effort="2.94" lower="-0.785" upper="0.785" velocity="5.24"/>
+    <limit effort="2.94" lower="-0.785" upper="0.785" velocity="4.71"/>
     <dynamics damping="0.05" friction="0.0"/>
   </joint>
@@ -129,5 +129,5 @@
     <origin rpy="0 0 0" xyz="-0.01744 0.0430692 0"/>
     <axis xyz="0 1 0"/>
-    <limit effort="2.94" lower="-1.57" upper="1.57" velocity="5.24"/>
+    <limit effort="2.94" lower="-1.57" upper="1.57" velocity="4.71"/>
     <dynamics damping="0.05" friction="0.0"/>
   </joint>
@@ -148,5 +148,5 @@
     <origin rpy="0 0 0" xyz="0.018944 0.03239997 -0.0999999"/>
     <axis xyz="0 1 0"/>
-    <limit effort="2.94" lower="-2.2" upper="1.57" velocity="5.24"/>
+    <limit effort="2.94" lower="-2.2" upper="1.57" velocity="4.71"/>
     <dynamics damping="0.05" friction="0.0"/>
   </joint>
@@ -173,5 +173,5 @@
     <origin rpy="0 0 0" xyz="0.108484 -0.0148092 0.00022176"/>
     <axis xyz="1 0 0"/>
-    <limit effort="2.94" lower="-0.785" upper="0.785" velocity="5.24"/>
+    <limit effort="2.94" lower="-0.785" upper="0.785" velocity="4.71"/>
     <dynamics damping="0.05" friction="0.0"/>
   </joint>
@@ -192,5 +192,5 @@
     <origin rpy="0 0 0" xyz="0.01744 -0.0430692 0"/>
     <axis xyz="0 1 0"/>
-    <limit effort="2.94" lower="-1.57" upper="1.57" velocity="5.24"/>
+    <limit effort="2.94" lower="-1.57" upper="1.57" velocity="4.71"/>
     <dynamics damping="0.05" friction="0.0"/>
   </joint>
@@ -211,5 +211,5 @@
     <origin rpy="0 0 0" xyz="0.0189441 -0.03239997 -0.0999999"/>
     <axis xyz="0 1 0"/>
-    <limit effort="2.94" lower="-2.2" upper="1.57" velocity="5.24"/>
+    <limit effort="2.94" lower="-2.2" upper="1.57" velocity="4.71"/>
     <dynamics damping="0.05" friction="0.0"/>
   </joint>
@@ -236,5 +236,5 @@
     <origin rpy="0 0 0" xyz="-0.108371 -0.01521 0.00022012"/>
     <axis xyz="1 0 0"/>
-    <limit effort="2.94" lower="-0.785" upper="0.785" velocity="5.24"/>
+    <limit effort="2.94" lower="-0.785" upper="0.785" velocity="4.71"/>
     <dynamics damping="0.05" friction="0.0"/>
   </joint>
@@ -255,5 +255,5 @@
     <origin rpy="0 0 0" xyz="-0.01744 -0.0430692 0"/>
     <axis xyz="0 1 0"/>
-    <limit effort="2.94" lower="-1.57" upper="1.57" velocity="5.24"/>
+    <limit effort="2.94" lower="-1.57" upper="1.57" velocity="4.71"/>
     <dynamics damping="0.05" friction="0.0"/>
   </joint>
@@ -274,5 +274,5 @@
     <origin rpy="0 0 0" xyz="0.0189441 -0.03239997 -0.0999999"/>
     <axis xyz="0 1 0"/>
-    <limit effort="2.94" lower="-2.2" upper="1.57" velocity="5.24"/>
+    <limit effort="2.94" lower="-2.2" upper="1.57" velocity="4.71"/>
     <dynamics damping="0.05" friction="0.0"/>
   </joint>
@@ -339,11 +339,16 @@
     <gazebo>
       <plugin filename="ign_ros2_control-system" name="ign_ros2_control::IgnitionROS2ControlPlugin">
+        <!-- position_proportional_gain (sim servo stiffness) lives in this yaml:
+             it is a node parameter on /gz_ros2_control, not an SDF tag. -->
         <parameters>$(find barq_bringup)/config/ros2_controllers.yaml</parameters>
       </plugin>
     </gazebo>
-    <gazebo reference="FL_tibia_link"><mu1>0.9</mu1><mu2>0.9</mu2></gazebo>
-    <gazebo reference="FR_tibia_link"><mu1>0.9</mu1><mu2>0.9</mu2></gazebo>
-    <gazebo reference="RL_tibia_link"><mu1>0.9</mu1><mu2>0.9</mu2></gazebo>
-    <gazebo reference="RR_tibia_link"><mu1>0.9</mu1><mu2>0.9</mu2></gazebo>
+    <!-- Foot-ground friction, sweepable for sim-to-real envelope mapping (D-018).
+         0.9 ~= printed TPU pad on wood/tile; the real value gets measured on hardware. -->
+    <xacro:arg name="foot_mu" default="0.9"/>
+    <gazebo reference="FL_tibia_link"><mu1>$(arg foot_mu)</mu1><mu2>$(arg foot_mu)</mu2></gazebo>
+    <gazebo reference="FR_tibia_link"><mu1>$(arg foot_mu)</mu1><mu2>$(arg foot_mu)</mu2></gazebo>
+    <gazebo reference="RL_tibia_link"><mu1>$(arg foot_mu)</mu1><mu2>$(arg foot_mu)</mu2></gazebo>
+    <gazebo reference="RR_tibia_link"><mu1>$(arg foot_mu)</mu1><mu2>$(arg foot_mu)</mu2></gazebo>
     <!-- 2D lidar (STL-27L-class: 360 deg, 25 m, 21.6 kHz -> 2160 samples @ 10 Hz).
          frame/topic chosen for zero-config parity with the real driver (frame 'laser', /scan). -->
